File: Lock (Eagle Project)/Lock.sch (EAGLE design)
At the start: 16 parts, among them T1 2N2222, T2 2N2222, T3 2N2222, U1 ARDUINOR3-BPLACE

Commit message: afsd
Parts:
- removed R1, R6: (no value), adafruit:R-US_R1005
- R2, R3: value (none) -> 220 ohms
- R4, R7: value (none) -> 1k ohms
- R5: value (none) -> 1k ohms; R5 (none) -> 1k
- renumbered BATT1 to 12V, LED2 to GREEN, LED3 to RED, U$1 to IR_RECIEVER, U$2 to BLUETOOTH
Connections:
- removed net N$10: IR_RECIEVER.GND, T1.E, T2.E, U1.GND1
- removed net N$11: R6.1, U1.D11
- removed net N$16: BLUETOOTH.+5V, U1.5V
- net N$1: now also R4.2; no longer R4.1
- net N$12: now also R4.1; no longer R4.2
- net N$17: now also IR_RECIEVER.GND
- net N$18: now also R7.2; no longer R7.1
- net N$20: now also T1.E, T2.E, U1.GND1
- net N$21: now also R7.1; no longer R7.2
- net N$3: now also U1.D11; no longer R6.2
- net N$4: now also BLUETOOTH.+5V, U1.5V; no longer R1.2
- net N$9: no longer R1.1
Other:
- moved on the sheet: R4, R7
